File: Week4/Clock/Clock.kicad_sch (KiCad schematic)
At the start: 41 parts, among them J1 PJ-102AH, J2 Conn_01x06, SW1 RotaryEncoder_Switch, SW2 Omron_B3F_SPST, U1 WH2004A-CFH-JT#, U2 ATmega328-PU, U3 L7805_TO92, U4 DS1307_DIP-8, U5 MAX7219, U6 MAX7219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

Commit message: Updated Schema & PCB
PCB was completely redone with only two DRC warnings which pertain to the Power In but nothing big, Changed to smaller LCD (Thankfully more space)
Parts:
- removed J1: PJ-102AH, footprints:PJ-102AH, symbol HPS:PJ-102AH
- removed U1: WH2004A-CFH-JT#, footprints:WH2004A-CFH-JT#, symbol HPS:WH2004A-CFH-JT#
- added DS1: TC1602A-01T, footprints:TC1602A-01T, symbol HPS:TC1602A-01T
- added J1: Power_inlet_vertical, footprints:Wurth-694106402002, symbol HPS:Power_inlet_vertical
- added R11: R_0805_1K, footprints:R_0805_2012Metric, symbol HPS:R_0805_1K
- SW1: footprint footprints:RotaryEncoder_Alps_EC11E-Switch_Vertical_H20mm_CircularMountingHoles -> footprints:RotaryEncoder_TT_EN11-Switch_Vertical_H20mm_CircularMountingHoles; Digikey PN (none) -> 987-1398-ND
Connections:
- net GND: now also DS1.1 (VSS), DS1.5 (R/W), J1.2 (OUT), R11.2
- net LCD D4: now also DS1.11 (D4)
- net LCD D5: now also DS1.12 (D5)
- net LCD D6: now also DS1.13 (D6)
- net LCD D7: now also DS1.14 (D7)
- net LCD E: now also DS1.6 (E)
- net LCD RS: now also DS1.4 (RS)
- net ROT ENC A OUT: now also R3.1, SW1.A
- net ROT ENC B OUT: now also R2.2, SW1.B
- net VCC: now also C10.1, C7.1, C8.1, C9.1, R6.1, R8.1, U5.19 (V+), U6.19 (V+), DS1.15 (LED(+)), DS1.2 (VDD)
- net at C2.1, U3.3 (VI): now also J1.1 (POLE)
- net at RV1.2: now also DS1.3 (VO)
- new net: DS1.16 (LED(-)), R11.1
Other:
- moved on the sheet: BT1, C1, C11, C2, C3, C4, C5, C6, J2, R1, R10, R2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
