File: Week6/Clock/Clock.kicad_pcb (KiCad board)
At the start: 2 copper layers, 140 x 90 mm, 63 parts, among them J1 Power_inlet_vertical, J2 Conn_01x06, SW1 RotaryEncoder_Switch, SW2 Omron_B3F_SPST, U1 L7805, U2 ATmega328-PU, U4 DS1307_DIP-8, U5 MAX7219, U6 MAX7219, Y1 Crystal 16MHZ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

Commit message: Image update
Parts:
- added G***: LOGO, Logo:Kirby, B.Cu at (146.0, 136.5)
