File: Clock CAD & Code/Clock/Clock.kicad_pcb (KiCad board)
At the start: 2 copper layers, 140 x 90 mm, 62 parts, among them J1 Power_inlet_vertical, J2 Conn_01x06, J3 Conn_02x03_Odd_Even, SW1 RotaryEncoder_Switch, SW2 Omron_B3F_SPST, U1 L7805, U2 ATmega328-PU, U4 DS1307_DIP-8, U5 MAX7219, U6 MAX7219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

Commit message: Fixed some more issues
Parts:
- removed C11: C_0805_0.1uf, footprints:C_0805_2012Metric
- J1: value Power_inlet_vertical -> PJ-102AH; footprint footprints:Wurth-694106402002 -> footprints:PJ-102AH
- moved R7 4.68 mm to (193.4, 122.0), turned to 180 degrees
- moved J1 1.35 mm to (203.0, 132.7)
Connections:
- SW2 pad 2: VCC -> ~{RST}
- SW2 pad 3: unconnected-(SW2-Pad3) -> GND
Routing:
- net GND: track 124.8 -> 111.6 mm, vias 18 -> 17
- net ~{RST}: track 61.3 -> 72.2 mm, vias 3 -> 5
- net Net-(C2-Pad1): track 5.37 -> 12.8 mm
- net Net-(D3-Pad2): track 9.22 -> 15.4 mm, vias 0 -> 2
- net SCK: track 142.7 -> 140.6 mm
- net LOAD MAX: track 184.6 -> 183.7 mm

Commit message: Gerber gerber
Parts:
- added C11: C_0805_0.1uf, footprints:C_0805_2012Metric, F.Cu at (190.2, 115.0)
- moved J1 1.70 mm to (201.9, 134.0), turned to -90 degrees
Connections:
- J2 pad 6: ~{RST} -> Net-(C11-Pad2)
Routing:
- net GND: track 111.6 -> 97.5 mm
- net VCC: track 87.1 -> 77.4 mm, vias 3 -> 2
- net ~{RST}: track 72.2 -> 75.8 mm
- net Net-(C11-Pad2): track 0.00 -> 2.85 mm
- net Net-(C2-Pad1): track 12.8 -> 12.1 mm
