File: Clock CAD & Code/Clock/Clock.kicad_sch (KiCad schematic)
At the start: 56 parts, among them J1 Power_inlet_vertical, J2 Conn_01x06, SW1 RotaryEncoder_Switch, SW2 Omron_B3F_SPST, U1 L7805, U2 ATmega328-PU, U4 DS1307_DIP-8, U5 MAX7219, U6 MAX7219, Y1 Crystal 16MHZ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

Commit message: Fixed DRC and ERC
Parts:
- removed R10: R_0805_10K, footprints:R_0805_2012Metric, symbol HPS:R_0805_10K
- removed R11, R14: R_0805_1K, footprints:R_0805_2012Metric, symbol HPS:R_0805_1K
- removed R7: R_0805_4.7K, footprints:R_0805_2012Metric, symbol HPS:R_0805_4.7K
- added J3: Conn_02x03_Odd_Even, footprints:PinHeader_2x03_P2.54mm_Vertical, symbol HPS:Conn_02x03_Odd_Even
- added R7: R_0805_2.2K, footprints:R_0805_2012Metric, symbol HPS:R_0805_2.2K
- C11: value 100n -> C_0805_0.1uf
Connections:
- net DATA MAX: now also U2.4 (INT0/PD2), U6.1 (DIN); no longer R4.1, R5.1, U2.17 (PB3), U5.12 (LOAD), U6.12 (LOAD)
- net GND: now also C11.2, DS1.16 (LED(-)), SW2.4 (B), J3.6 (Pin_6)
- net LCD E: now also J3.1 (Pin_1)
- net LOAD MAX: now also R4.1, R5.1, U2.17 (MOSI/PB3), U5.12 (LOAD), U6.12 (LOAD), J3.4 (Pin_4); no longer U2.4 (PD2), U6.1 (DIN)
- net SCK: now also J3.3 (Pin_3), R7.1
- net VCC: now also J3.2 (Pin_2)
- net ~{RST}: now also J2.6 (Pin_6), SW2.1 (A), J3.5 (Pin_5)
- net at D3.2 (A): now also R7.2
- net at R6.2: now also U5.18 (ISET)
- net VBAT: no longer names the net of BT1.1 (+), U4.3 (VBAT), VBAT_TP1.1
- removed net ~{RESET BTN}: C11.2, J2.6 (Pin_6), SW2.1 (A)
- no-connect marks 2 -> 12
Other:
- note added: "ICSP"
- moved on the sheet: A_TP1, B_TP1, C12, J2, R2, R3, R9, RX_TP1, SW1, SW2, TX_TP1

Commit message: Fixed some more issues
Parts:
- removed C11: C_0805_0.1uf, footprints:C_0805_2012Metric, symbol HPS:C_0805_0.1uf
Connections:
- net GND: now also SW2.3 (B)
- net VCC: no longer SW2.2 (A)
- net ~{RST}: now also SW2.2 (A)
- no-connect marks 12 -> 11
Changed lines of the file:
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@@
   (junction (at 170.18 170.18) (diameter 0) (color 0 0 0 0)
   )
-  (junction (at 180.34 41.91) (diameter 0) (color 0 0 0 0)
-  )
   (junction (at 49.53 228.6) (diameter 0) (color 0 0 0 0)
   )
@@
   (junction (at 40.64 43.18) (diameter 0) (color 0 0 0 0)
   )
+  (junction (at 182.88 27.94) (diameter 0) (color 0 0 0 0)
+  )
   (junction (at 69.85 30.48) (diameter 0) (color 0 0 0 0)
   )
@@
   (junction (at 182.88 226.06) (diameter 0) (color 0 0 0 0)
   )
+  (junction (at 180.34 40.64) (diameter 0) (color 0 0 0 0)
+  )
   (junction (at 184.15 161.29) (diameter 0) (color 0 0 0 0)
   )
@@
   (no_connect (at 34.29 99.06))
   (no_connect (at 34.29 96.52))
-  (no_connect (at 180.34 27.94))
   (no_connect (at 130.81 40.64))
   (no_connect (at 34.29 91.44))
@@
     (stroke (width 0) (type default) (color 0 0 0 0))
   )
+  (wire (pts (xy 180.34 27.94) (xy 182.88 27.94))
+    (stroke (width 0) (type default) (color 0 0 0 0))
+  )
+  (wire (pts (xy 180.34 40.64) (xy 180.34 58.42))
+    (stroke (width 0) (type default) (color 0 0 0 0))
+  )
   (wire (pts (xy 317.5 120.65) (xy 317.5 124.46))
     (stroke (width 0) (type default) (color 0 0 0 0))
@@
     (stroke (width 0) (type default) (color 0 0 0 0))
   )
+  (wire (pts (xy 182.88 38.1) (xy 182.88 40.64))
+    (stroke (width 0) (type default) (color 0 0 0 0))
+  )
   (wire (pts (xy 204.47 187.96) (xy 204.47 167.64))
     (stroke (width 0) (type default) (color 0 0 0 0))
@@
     (stroke (width 0) (type default) (color 0 0 0 0))
   )
-  (wire (pts (xy 180.34 38.1) (xy 180.34 41.91))
+  (wire (pts (xy 180.34 38.1) (xy 180.34 40.64))
     (stroke (width 0) (type default) (color 0 0 0 0))
   )
@@
     (stroke (width 0) (type default) (color 0 0 0 0))
   )
-  (wire (pts (xy 189.23 41.91) (xy 187.96 41.91))
-    (stroke (width 0) (type default) (color 0 0 0 0))
-  )
   (wire (pts (xy 207.01 151.13) (xy 207.01 135.89))
     (stroke (width 0) (type default) (color 0 0 0 0))
@@
     (stroke (width 0) (type default) (color 0 0 0 0))
   )
+  (wire (pts (xy 182.88 40.64) (xy 180.34 40.64))
+    (stroke (width 0) (type default) (color 0 0 0 0))
+  )
   (wire (pts (xy 58.42 43.18) (xy 69.85 43.18))
     (stroke (width 0) (type default) (color 0 0 0 0))
@@
     (stroke (width 0) (type default) (color 0 0 0 0))
   )
-  (wire (pts (xy 180.34 41.91) (xy 180.34 58.42))
-    (stroke (width 0) (type default) (color 0 0 0 0))
-  )
   (polyline (pts (xy 344.17 95.25) (xy 344.17 137.16))
     (stroke (width 0) (type default) (color 0 0 0 0))
@@
     (pin "1")
   )
-  (symbol (lib_id "HPS:GND") (at 189.23 41.91 90) (unit 1)
-    (in_bom yes) (on_board yes) (fields_autoplaced)
-    (property "Reference" "#PWR0110" (id 0) (at 195.58 41.91 0)
-      (effects (font (size 1.27 1.27)) hide)
-    )
-    (property "Value" "GND" (id 1) (at 193.9544 41.91 0))
-    (property "Footprint" "" (id 2) (at 189.23 41.91 0)
-      (effects (font (size 1.27 1.27)) hide)
-    )
-    (property "Datasheet" "" (id 3) (at 189.23 41.91 0)
-      (effects (font (size 1.27 1.27)) hide)
-    )
-    (pin "1")
-  )
   (symbol (lib_id "HPS:VCC") (at 72.39 184.15 0) (unit 1)
     (in_bom yes) (on_board yes) (fields_autoplaced)
@@
     (pin "1")
   )
-  (symbol (lib_id "HPS:C_0805_0.1uf") (at 184.15 41.91 90) (unit 1)
-    (in_bom yes) (on_board yes) (fields_autoplaced)
-    (property "Reference" "C11" (id 0) (at 182.8799 38.1 0)
-      (effects (font (size 1.27 1.27)) (justify left))
-    )
-    (property "Value" "C_0805_0.1uf" (id 1) (at 185.4199 38.1 0)
-      (effects (font (size 1.27 1.27)) (justify left))
-    )
-    (property "Footprint" "footprints:C_0805_2012Metric" (id 2) (at 187.96 40.9448 0)
-      (effects (font (size 1.27 1.27)) hide)
-    )
-    (property "Datasheet" "https://datasheets.avx.com/X7RDielectric.pdf" (id 3) (at 181.61 41.275 0)
-      (effects (font (size 1.27 1.27)) hide)
-    )
-    (property "MFG" "AVX Corporation" (id 4) (at 190.5 41.91 0)
-      (effects (font (size 1.27 1.27)) hide)
-    )
-    (property "MPN" "08055C104KAT2A" (id 5) (at 193.04 41.91 0)
-      (effects (font (size 1.27 1.27)) hide)
-    )
-    (property "Digikey PN" "478-1395-1-ND" (id 6) (at 198.12 41.91 0)
-      (effects (font (size 1.27 1.27)) hide)
-    )
-    (property "Mouser PN" "N/A" (id 7) (at 200.66 41.91 0)
-      (effects (font (size 1.27 1.27)) hide)
-    )
-    (property "Voltage" "N/A" (id 8) (at 203.2 41.91 0)
-      (effects (font (size 1.27 1.27)) hide)
-    )
-    (property "Dielectric" "N/A" (id 9) (at 203.2 41.91 0)
-      (effects (font (size 1.27 1.27)) hide)
-    )
-    (property "Tolerance" "N/A" (id 10) (at 203.2 41.91 0)
-      (effects (font (size 1.27 1.27)) hide)
-    )
-    (pin "1")
-    (pin "2")
-  )
   (symbol (lib_id "HPS:VCC") (at 279.4 104.14 0) (unit 1)
     (in_bom yes) (on_board yes)
@@
     (pin "2")
   )
-  (symbol (lib_id "HPS:VCC") (at 182.88 38.1 270) (unit 1)
-    (in_bom yes) (on_board yes) (fields_autoplaced)
-    (property "Reference" "#PWR01" (id 0) (at 179.07 38.1 0)
-      (effects (font (size 1.27 1.27)) hide)
-    )
-    (property "Value" "VCC" (id 1) (at 187.5536 38.1 0))
-    (property "Footprint" "" (id 2) (at 182.88 38.1 0)
-      (effects (font (size 1.27 1.27)) hide)
-    )
-    (property "Datasheet" "" (id 3) (at 182.88 38.1 0)
-      (effects (font (size 1.27 1.27)) hide)
-    )
-    (pin "1")
-  )
   (symbol (lib_id "HPS:GND") (at 57.15 100.33 0) (unit 1)
     (in_bom yes) (on_board yes) (fields_autoplaced)
@@
       (reference "#G2") (unit 1) (value "LOGO") (footprint "")
     )
-    (path "/fb4d5b8c-776c-40ea-804f-0ca9c5d8e8fe"
-      (reference "#PWR01") (unit 1) (value "VCC") (footprint "")
-    )
     (path "/dc1683e1-9605-46e6-8cde-cee330b30c22"
       (reference "#PWR02") (unit 1) (value "GND") (footprint "")
@@
       (reference "#PWR0109") (unit 1) (value "GND") (footprint "")
     )
-    (path "/10786c67-8496-465e-83af-0e7ac2fea39d"
-      (reference "#PWR0110") (unit 1) (value "GND") (footprint "")
-    )
     (path "/914de20c-a312-47aa-a6f3-9f8c7b1b0679"
       (reference "#PWR0111") (unit 1) (value "VCC") (footprint "")
@@
       (reference "C10") (unit 1) (value "C_0805_0.1uf") (footprint "footprints:C_0805_2012Metric")
     )
-    (path "/e69f6b4f-1c99-4a63-9c93-5458acaca919"
-      (reference "C11") (unit 1) (value "C_0805_0.1uf") (footprint "footprints:C_0805_2012Metric")
-    )
     (path "/17f5096d-2fc7-45f7-9fd9-de75c2f2839d"

Commit message: Gerber gerber
Parts:
- removed J1: Power_inlet_vertical, footprints:Wurth-694106402002, symbol HPS:Power_inlet_vertical
- added C11: C_0805_0.1uf, footprints:C_0805_2012Metric, symbol HPS:C_0805_0.1uf
- added J1: PJ-102AH, footprints:PJ-102AH, symbol HPS:PJ-102AH
Connections:
- net GND: now also J1.2 (OUT)
- net ~{RST}: now also C11.1; no longer J2.6 (Pin_6)
- net at C2.1, U1.1 (IN): now also J1.1 (POLE)
- new net: C11.2, J2.6 (Pin_6)
Changed lines of the file:
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@@
     (stroke (width 0) (type default) (color 0 0 0 0))
   )
-  (wire (pts (xy 180.34 40.64) (xy 180.34 58.42))
-    (stroke (width 0) (type default) (color 0 0 0 0))
-  )
   (wire (pts (xy 317.5 120.65) (xy 317.5 124.46))
     (stroke (width 0) (type default) (color 0 0 0 0))
@@
     (stroke (width 0) (type default) (color 0 0 0 0))
   )
+  (wire (pts (xy 180.34 40.64) (xy 180.34 58.42))
+    (stroke (width 0) (type default) (color 0 0 0 0))
+  )
   (wire (pts (xy 52.07 138.43) (xy 52.07 142.24))
     (stroke (width 0) (type default) (color 0 0 0 0))
@@
     (stroke (width 0) (type default) (color 0 0 0 0))
   )
+  (wire (pts (xy 209.55 67.31) (xy 212.09 67.31))
+    (stroke (width 0) (type default) (color 0 0 0 0))
+  )
   (wire (pts (xy 208.28 133.35) (xy 208.28 149.86))
     (stroke (width 0) (type default) (color 0 0 0 0))
@@
     (stroke (width 0) (type default) (color 0 0 0 0))
   )
+  (wire (pts (xy 195.58 67.31) (xy 201.93 67.31))
+    (stroke (width 0) (type default) (color 0 0 0 0))
+  )
   (polyline (pts (xy 85.09 15.24) (xy 85.09 64.77))
     (stroke (width 0) (type default) (color 0 0 0 0))
@@
     (stroke (width 0) (type default) (color 0 0 0 0))
   )
-  (wire (pts (xy 212.09 67.31) (xy 195.58 67.31))
-    (stroke (width 0) (type default) (color 0 0 0 0))
-  )
   (wire (pts (xy 67.31 157.48) (xy 71.12 157.48))
     (stroke (width 0) (type default) (color 0 0 0 0))
@@
     (effects (font (size 1.27 1.27) bold) (justify left bottom))
   )
-  (text "Reset Button\n" (at 191.262 55.6768 90)
+  (text "Reset Button\n" (at 205.74 50.8 90)
     (effects (font (size 1.27 1.27) bold) (justify left bottom))
   )
@@
     (pin "1")
   )
+  (symbol (lib_id "HPS:PJ-102AH") (at 29.21 33.02 0) (unit 1)
+    (in_bom yes) (on_board yes) (fields_autoplaced)
+    (property "Reference" "J1" (id 0) (at 26.67 20.32 0)
+      (effects (font (size 1.524 1.524)))
+    )
+    (property "Value" "PJ-102AH" (id 1) (at 26.67 24.13 0)
+      (effects (font (size 1.524 1.524)))
+    )
+    (property "Footprint" "footprints:PJ-102AH" (id 2) (at 26.67 27.94 0)
+      (effects (font (size 1.524 1.524)))
+    )
+    (property "Datasheet" "https://www.cuidevices.com/product/resource/pj-102ah.pdf" (id 3) (at 30.734 44.958 0)
+      (effects (font (size 1.524 1.524)) hide)
+    )
+    (property "MFG" "CUI Devices" (id 4) (at 29.21 50.8 0)
+      (effects (font (size 1.27 1.27)) hide)
+    )
+    (property "MPN" "PJ-102AH" (id 5) (at 29.21 53.34 0)
+      (effects (font (size 1.27 1.27)) hide)
+    )
+    (property "Digikey PN" "CP-102AH-ND" (id 6) (at 30.734 58.547 0)
+      (effects (font (size 1.27 1.27)) hide)
+    )
+    (property "Mouser PN" "490-PJ-102AH" (id 7) (at 29.21 55.753 0)
+      (effects (font (size 1.27 1.27)) hide)
+    )
+    (pin "1")
+    (pin "2")
+    (pin "3")
+  )
   (symbol (lib_id "HPS:L7805") (at 58.42 30.48 0) (unit 1)
     (in_bom yes) (on_board yes) (fields_autoplaced)
@@
     (pin "1")
   )
-  (symbol (lib_id "HPS:Power_inlet_vertical") (at 29.21 33.02 0) (unit 1)
-    (in_bom yes) (on_board yes)
-    (property "Reference" "J1" (id 0) (at 26.67 20.32 0)
-      (effects (font (size 1.524 1.524)))
-    )
-    (property "Value" "Power_inlet_vertical" (id 1) (at 26.67 24.13 0)
-      (effects (font (size 1.524 1.524)))
-    )
-    (property "Footprint" "footprints:Wurth-694106402002" (id 2) (at 19.05 34.29 90)
-      (effects (font (size 1.524 1.524)))
-    )
-    (property "Datasheet" "https://www.we-online.com/katalog/datasheet/6941xx402002.pdf" (id 3) (at 30.734 44.958 0)
-      (effects (font (size 1.524 1.524)) hide)
-    )
-    (property "MFG" "Wurth" (id 4) (at 29.21 50.8 0)
-      (effects (font (size 1.27 1.27)) hide)
-    )
-    (property "MPN" "694106402002" (id 5) (at 29.21 53.34 0)
-      (effects (font (size 1.27 1.27)) hide)
-    )
-    (property "Digikey PN" "732-5931-ND" (id 6) (at 30.734 58.547 0)
-      (effects (font (size 1.27 1.27)) hide)
-    )
-    (pin "1")
-    (pin "2")
-    (pin "3")
-  )
   (symbol (lib_id "HPS:Conn_01x06") (at 217.17 59.69 0) (unit 1)
     (in_bom yes) (on_board yes)
@@
     (pin "1")
   )
+  (symbol (lib_id "HPS:C_0805_0.1uf") (at 205.74 67.31 90) (unit 1)
+    (in_bom yes) (on_board yes) (fields_autoplaced)
+    (property "Reference" "C11" (id 0) (at 205.74 59.69 90))
+    (property "Value" "C_0805_0.1uf" (id 1) (at 205.74 62.23 90))
+    (property "Footprint" "footprints:C_0805_2012Metric" (id 2) (at 209.55 66.3448 0)
+      (effects (font (size 1.27 1.27)) hide)
+    )
+    (property "Datasheet" "https://datasheets.avx.com/X7RDielectric.pdf" (id 3) (at 203.2 66.675 0)
+      (effects (font (size 1.27 1.27)) hide)
+    )
+    (property "MFG" "AVX Corporation" (id 4) (at 212.09 67.31 0)
+      (effects (font (size 1.27 1.27)) hide)
+    )
+    (property "MPN" "08055C104KAT2A" (id 5) (at 214.63 67.31 0)
+      (effects (font (size 1.27 1.27)) hide)
+    )
+    (property "Digikey PN" "478-1395-1-ND" (id 6) (at 219.71 67.31 0)
+      (effects (font (size 1.27 1.27)) hide)
+    )
+    (property "Mouser PN" "N/A" (id 7) (at 222.25 67.31 0)
+      (effects (font (size 1.27 1.27)) hide)
+    )
+    (property "Voltage" "N/A" (id 8) (at 224.79 67.31 0)
+      (effects (font (size 1.27 1.27)) hide)
+    )
+    (property "Dielectric" "N/A" (id 9) (at 224.79 67.31 0)
+      (effects (font (size 1.27 1.27)) hide)
+    )
+    (property "Tolerance" "N/A" (id 10) (at 224.79 67.31 0)
+      (effects (font (size 1.27 1.27)) hide)
+    )
+    (pin "1")
+    (pin "2")
+  )
   (symbol (lib_id "HPS:VCC") (at 52.07 138.43 0) (unit 1)
     (in_bom yes) (on_board yes) (fields_autoplaced)
@@
       (reference "C10") (unit 1) (value "C_0805_0.1uf") (footprint "footprints:C_0805_2012Metric")
     )
+    (path "/62f026f3-2ade-4ab6-9971-a851915086a9"
+      (reference "C11") (unit 1) (value "C_0805_0.1uf") (footprint "footprints:C_0805_2012Metric")
+    )
     (path "/17f5096d-2fc7-45f7-9fd9-de75c2f2839d"
       (reference "C12") (unit 1) (value "C_0805_1uf") (footprint "footprints:C_0805_2012Metric")
@@
       (reference "H4") (unit 1) (value "MountingHole") (footprint "footprints:MountingHole_3.2mm_M3")
     )
-    (path "/51816d45-b9e2-4280-b65a-6b8bbbd817b1"
-      (reference "J1") (unit 1) (value "Power_inlet_vertical") (footprint "footprints:Wurth-694106402002")
+    (path "/20fd1c10-b75b-400d-af01-250347676ba7"
+      (reference "J1") (unit 1) (value "PJ-102AH") (footprint "footprints:PJ-102AH")
     )
     (path "/5912c6e4-f0ee-4e45-b4cb-e87568483e9f"
